File: rear-mcu/rear-mcu.kicad_pcb (KiCad board)
At the start: 2 copper layers, 30 x 50 mm, 54 parts, among them J1 Conn_02x10_Odd_Even, J2 USB_C_Receptacle_USB2.0_16P, SW1 SW_SPST, U1 STM32F103C8Tx, U2 SN65HVD256D, U3 AP2204K-ADJ, U4 AP2204K-ADJ, Y1 8M, Y2 32.768k

Commit message: layout
Parts:
- R10, U2: moved to B.Cu
- moved C8 65.9 mm to (121.0, 101.0)
- moved C2 61.2 mm to (116.0, 96.0), turned to 90 degrees
- moved C9 60.1 mm to (117.5, 101.0)
- moved C3 55.1 mm to (109.8, 99.0), turned to -90 degrees
- moved U2 43.0 mm to (117.8, 120.2)
- moved R11 41.3 mm to (98.2, 113.7), turned to 90 degrees
- moved R10 38.7 mm to (100.8, 113.3), turned to -90 degrees
- moved Y2 29.9 mm to (119.5, 98.0), turned to 90 degrees
- moved Y1 22.9 mm to (112.9, 97.5), turned to 180 degrees
- moved J2 2.75 mm to (115.8, 129.2)
- moved C5 1.12 mm to (120.0, 104.0)
- moved C4 1.12 mm to (121.8, 104.0)
- moved C17 1.01 mm to (113.0, 102.8)
- moved C6 0.96 mm to (121.8, 107.3)
- moved U1 0.96 mm to (115.2, 109.0)
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Connections:
- C10 pad 1: +3V3 -> +3.3V
- C17 pad 1: +3V3 -> +3.3V
- C4 pad 1: +3V3 -> +3.3V
- C5 pad 1: +3V3 -> +3.3V
- C6 pad 1: +3V3 -> +3.3V
- C7 pad 1: +3V3 -> +3.3V
- J1 pad 10: BMS_signal -> BSPD_signal1
- J1 pad 11: SWDIO -> SWDCLK
- J1 pad 12: IMD_signal -> BSPD_signal2
- J1 pad 13: SWDCLK -> SWDIO
- J1 pad 14: BSPD_signal -> BSPD_signal3
- J1 pad 16: BSPD_signal1 -> unconnected-(J1-Pin_16-Pad16)
- J1 pad 18: BSPD_signal2 -> CAN-
- J1 pad 20: BSPD_signal3 -> CAN+
- J1 pad 4: CAN+ -> BMS_signal
- J1 pad 6: CAN- -> IMD_signal
- J1 pad 8: unconnected-(J1-Pin_8-Pad8) -> BSPD_signal
- U1 pad 32: /CAN_TX -> USB_D-
- U1 pad 33: /CAN_RX -> USB_D+
- U1 pad 45: unconnected-(U1-PB8-Pad45) -> CAN_TX
- U1 pad 46: unconnected-(U1-PB9-Pad46) -> CAN_RX
- U2 pad 1: /CAN_TX -> CAN_TX
- U2 pad 4: /CAN_RX -> CAN_RX
- U2 pad 5: +3V3 -> +3.3V
Routing:
- net +5V: track 0.00 -> 82.9 mm, vias 0 -> 3
- net +3.3V: track 0.00 -> 55.8 mm
- net BMS_signal: track 0.00 -> 45.8 mm
- net BSPD_signal3: track 0.00 -> 43.5 mm
- net BSPD_signal2: track 0.00 -> 43.4 mm
- net IMD_signal: track 0.00 -> 41.3 mm
- net BSPD_signal1: track 0.00 -> 41.2 mm
- net BSPD_signal: track 0.00 -> 41.2 mm
- net /RESET: track 0.00 -> 26.8 mm, vias 0 -> 2
- net CAN_TX: track 0.00 -> 20.3 mm, vias 0 -> 1
- net SWDIO: track 0.00 -> 15.1 mm
- net USB_D+: track 0.00 -> 14.7 mm
- net CAN_RX: track 0.00 -> 14.3 mm, vias 0 -> 1
- net VDC: track 0.00 -> 14.3 mm
- net USB_D-: track 0.00 -> 13.7 mm
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
Commit message: layout
Parts:
- R12, R14, R16: moved to B.Cu
- moved R12 47.9 mm to (106.2, 116.8)
- moved R13 46.5 mm to (106.2, 116.8), turned to 180 degrees
- moved R14 44.5 mm to (106.4, 115.0)
- moved R15 43.4 mm to (106.4, 115.0), turned to 180 degrees
- moved R16 41.4 mm to (106.4, 112.2), turned to -90 degrees
- moved R17 40.6 mm to (106.4, 112.2), turned to 90 degrees
- moved R20 40.6 mm to (101.8, 115.6), turned to 90 degrees
- moved R11 11.3 mm to (106.2, 121.8), turned to -90 degrees
- moved R10 7.17 mm to (104.6, 119.4)
- moved C10 1.12 mm to (110.6, 114.0), turned to -90 degrees
Connections:
- R10 pad 2: /BMS_LED -> BMS_LED
- R11 pad 1: /BMS_LED -> BMS_LED
- R12 pad 2: /IMD_LED -> IMD_LED
- R13 pad 1: /IMD_LED -> IMD_LED
- R14 pad 2: /BSPD_LED -> BSPD_LED
- R15 pad 1: /BSPD_LED -> BSPD_LED
- R16 pad 2: /BSPD_Check1 -> BSPD_Check1
- R17 pad 1: /BSPD_Check1 -> BSPD_Check1
- R18 pad 2: /BSPD_Check2 -> BSPD_Check2
- R19 pad 1: /BSPD_Check2 -> BSPD_Check2
- R20 pad 2: /BSPD_Check3 -> BSPD_Check3
- R21 pad 1: /BSPD_Check3 -> BSPD_Check3
- U1 pad 13: /BMS_LED -> SW_signal
- U1 pad 14: /IMD_LED -> BSPD_Check3
- U1 pad 15: /BSPD_LED -> BSPD_Check2
- U1 pad 16: SW_signal -> BSPD_Check1
- U1 pad 18: /BSPD_Check1 -> BSPD_LED
- U1 pad 19: /BSPD_Check2 -> IMD_LED
- U1 pad 21: /BSPD_Check3 -> BMS_LED
Routing:
- net BMS_LED: track 0.00 -> 15.3 mm, vias 0 -> 1
- net IMD_signal: track 41.3 -> 52.9 mm
- net BSPD_signal: track 41.2 -> 52.5 mm
- net IMD_LED: track 0.00 -> 10.4 mm, vias 0 -> 1
- net BSPD_signal1: track 41.2 -> 50.3 mm
- net BSPD_Check1: track 0.00 -> 8.39 mm, vias 0 -> 1
- net BSPD_LED: track 0.00 -> 8.34 mm, vias 0 -> 1
- net BMS_signal: track 45.8 -> 53.8 mm
- net BSPD_signal3: track 43.5 -> 36.5 mm

Commit message: finish layout
Parts:
- added C11: 100n, Capacitor_SMD:C_0603_1608Metric, B.Cu at (113.0, 118.8)
- added G***: LOGO, logo:galaxy_logo_10mm, F.Cu at (116.0, 121.8)
- added G***: LOGO, logo:nckufs_logo_10mm, F.Cu at (116.5, 117.0)
- added G***: LOGO, logo:fire_shark_4mm, F.Cu at (106.2, 92.5)
- added G***: LOGO, logo:fire_shark_logo_20mm, B.Cu at (114.2, 100.2)
- C1: value 0.1u -> 100n; moved to B.Cu
- R18, R20, R22, R23, R24, R25, R3, R5: moved to B.Cu
- moved C1 71.0 mm to (119.5, 116.5), turned to 180 degrees
- moved C16 69.3 mm to (124.5, 119.5), turned to -90 degrees
- moved R4 66.0 mm to (123.6, 115.5), turned to 180 degrees
- moved R5 65.1 mm to (123.7, 115.5)
- moved R3 64.9 mm to (123.4, 110.5)
- moved R1 64.8 mm to (123.3, 110.5), turned to 180 degrees
- moved R22 58.5 mm to (122.8, 121.7), turned to -90 degrees
- moved R23 56.1 mm to (122.8, 118.5), turned to -90 degrees
- moved R2 55.4 mm to (112.7, 89.5), turned to 180 degrees
- moved R25 53.7 mm to (117.5, 128.7), turned to -90 degrees
- moved R24 52.5 mm to (114.5, 128.7), turned to -90 degrees
- moved R19 41.7 mm to (106.8, 108.2), turned to 90 degrees
- moved R18 39.8 mm to (106.8, 108.2), turned to -90 degrees
- moved R21 38.3 mm to (107.2, 104.6), turned to 90 degrees
- moved R20 12.3 mm to (107.2, 104.6), turned to -90 degrees
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Connections:
- net Brake_signal renamed Brake_signal1
- net Current_signal renamed Brake_signal2
- C1 pad 1: GND -> +3.3V
- C1 pad 2: +3.3V -> GND
Routing:
- net +3.3V: track 55.8 -> 122.9 mm, vias 0 -> 7
- net SW_signal: track 0.00 -> 31.6 mm, vias 0 -> 2
- net GND: track 0.00 -> 25.4 mm, vias 0 -> 10
- net /ADC_IN1: track 0.00 -> 19.6 mm, vias 0 -> 2
- net Brake_signal2: track 0.00 -> 16.1 mm
- net /ADC_IN0: track 0.00 -> 14.7 mm, vias 0 -> 2
- net Brake_signal1: track 0.00 -> 9.68 mm
- net BSPD_signal3: track 36.5 -> 45.3 mm
- net +5V: track 82.9 -> 91.6 mm, vias 3 -> 4
- net Net-(C16-Pad1): track 0.00 -> 7.26 mm, vias 0 -> 2
- net BSPD_Check2: track 0.00 -> 5.01 mm, vias 0 -> 1
- net /RESET: track 26.8 -> 31.2 mm
- net BSPD_Check3: track 0.00 -> 4.45 mm, vias 0 -> 1
- net BSPD_signal2: track 43.4 -> 47.7 mm
- net Net-(J2-CC2): track 0.00 -> 2.64 mm, vias 0 -> 1
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- added copper zone on B.Cu, net GND
- added copper zone on F.Cu, net GND
Other:
- board text added: "rear MCU 2025.3 ver1.0"

Commit message: add: TSSI modify: CAN
Parts:
- added R26: 47k, Resistor_SMD:R_0603_1608Metric, B.Cu at (124.5, 112.2)
- moved C5 7.53 mm to (113.0, 101.2), turned to 180 degrees
- moved C8 1.80 mm to (122.5, 100.0), turned to -90 degrees
- moved Y1 1.19 mm to (112.2, 96.5)
- moved C3 1.12 mm to (109.2, 98.0)
- moved C2 0.77 mm to (116.2, 95.2), turned to 0 degrees
- moved R1 0.75 mm to (123.3, 109.8)
- moved R3 0.75 mm to (123.4, 109.8)
- moved C9 0.72 mm to (118.2, 101.0), turned to 180 degrees
- moved Y2 0.25 mm to (119.8, 98.0)
- moved R23 0.17 mm to (122.8, 118.7)
- moved R22 0.15 mm to (122.8, 121.8)
Connections:
- J1 pad 16: unconnected-(J1-Pin_16-Pad16) -> TSSI
- U1 pad 39: unconnected-(U1-PB3-Pad39) -> TSSI
- U1 pad 45: CAN_TX -> CAN_RX
- U1 pad 46: CAN_RX -> CAN_TX
Routing:
- net TSSI: track 0.00 -> 13.4 mm, vias 0 -> 1
- net GND: track 25.4 -> 36.0 mm, vias 10 -> 8
- net /LSE_IN: track 7.10 -> 10.3 mm
- net +3.3V: track 122.9 -> 125.1 mm
- net /HSE_OUT: track 10.3 -> 12.2 mm
- net /LSE_OUT: track 11.0 -> 9.29 mm
- net SW_signal: track 31.6 -> 33.2 mm
- net /HSE_IN: track 10.8 -> 12.4 mm
- net /RESET: track 31.2 -> 32.3 mm
- net CAN_RX: track 14.1 -> 13.1 mm
- net Brake_signal1: track 9.68 -> 8.93 mm
- net /ADC_IN0: track 14.7 -> 14.0 mm
- net Net-(C16-Pad1): track 7.26 -> 7.76 mm

Commit message: v2025.5
Parts:
- removed R4: 47k, Resistor_SMD:R_0603_1608Metric
- removed R5: 100k, Resistor_SMD:R_0603_1608Metric
- moved R1 3.22 mm to (124.5, 106.8), turned to -90 degrees
- moved R3 0.49 mm to (123.0, 109.5), turned to 180 degrees
Connections:
- net BMS_signal renamed BMS_Fault
- net BSPD_signal renamed BSPD_Fault
- net Brake_signal1 renamed BSPD_signal4
- net IMD_signal renamed IMD_Fault
- J1 pad 9: Brake_signal2 -> unconnected-(J1-Pin_9-Pad9)
- R1 pad 2: /ADC_IN0 -> BSPD_Check4
- R3 pad 1: /ADC_IN0 -> BSPD_Check4
- U1 pad 10: /ADC_IN0 -> unconnected-(U1-PA0-Pad10)
- U1 pad 17: unconnected-(U1-PA7-Pad17) -> BSPD_Check4
Routing:
- net /ADC_IN1: track 19.6 -> 0.00 mm, vias 2 -> 0
- net BSPD_Check4: track 0.00 -> 17.3 mm, vias 0 -> 3
- net Brake_signal2: track 16.1 -> 0.00 mm
- net /ADC_IN0: track 14.0 -> 0.00 mm, vias 2 -> 0
- net BSPD_signal4: track 8.93 -> 6.18 mm
- net GND: track 36.0 -> 35.2 mm, vias 8 -> 11
- net +5V: track 91.6 -> 92.2 mm
Other:
- board text added: "rear MCU v2025.5"
- board text removed: "rear MCU 2025.3 ver1.0"
