File: rear-mcu/rear-mcu.kicad_sch (KiCad schematic)
At the start: 55 parts, among them J1 Conn_02x10_Odd_Even, J2 USB_C_Receptacle_USB2.0_16P, SW1 SW_SPST, U1 STM32F103C8Tx, U2 SN65HVD256D, U3 AP2204K-ADJ, U4 AP2204K-ADJ, Y1 8M, Y2 32.768k

Commit message: add: TSSI modify: CAN
Parts:
- added R26: 47k, Resistor_SMD:R_0603_1608Metric, symbol Device:R
Connections:
- net CAN_RX: now also U1.45 (PB8); no longer U1.46 (PB9)
- net CAN_TX: now also U1.46 (PB9); no longer U1.45 (PB8)
- net GND: now also R26.2
- net TSSI: now reaches J1.16 (Pin_16)
- net TSSI: now also U1.39 (PB3), R26.1
- no-connect marks 21 -> 20
Changed lines of the file:
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@@
   (no_connect (at 168.91 71.12))
   (no_connect (at 135.89 91.44))
-  (no_connect (at 135.89 83.82))
   (no_connect (at 168.91 86.36))
   (no_connect (at 135.89 81.28))
@@
     (stroke (width 0) (type default))
   )
+  (wire (pts (xy 107.95 123.19) (xy 107.95 124.46))
+    (stroke (width 0) (type default))
+  )
   (wire (pts (xy 101.6 190.5) (xy 115.57 190.5))
     (stroke (width 0) (type default))
@@
     (stroke (width 0) (type default))
   )
+  (wire (pts (xy 107.95 114.3) (xy 107.95 115.57))
+    (stroke (width 0) (type default))
+  )
   (wire (pts (xy 153.67 124.46) (xy 151.13 124.46))
     (stroke (width 0) (type default))
@@
     )
   )
+  (global_label "TSSI" (shape input) (at 135.89 83.82 180) (fields_autoplaced)
+    (effects (font (size 1.27 1.27)) (justify right))
+    (property "Intersheetrefs" "${INTERSHEET_REFS}" (at 128.9134 83.82 0)
+      (effects (font (size 1.27 1.27)) (justify right) hide)
+    )
+  )
   (global_label "BSPD_signal" (shape input) (at 53.34 172.72 0) (fields_autoplaced)
     (effects (font (size 1.27 1.27)) (justify left))
@@
     )
   )
+  (global_label "CAN_TX" (shape input) (at 135.89 99.06 180) (fields_autoplaced)
+    (effects (font (size 1.27 1.27)) (justify right))
+    (property "Intersheetrefs" "${INTERSHEET_REFS}" (at 126.071 99.06 0)
+      (effects (font (size 1.27 1.27)) (justify right) hide)
+    )
+  )
   (global_label "CAN+" (shape input) (at 53.34 187.96 0) (fields_autoplaced)
     (effects (font (size 1.27 1.27)) (justify left))
@@
     )
   )
-  (global_label "CAN_TX" (shape input) (at 135.89 96.52 180) (fields_autoplaced)
-    (effects (font (size 1.27 1.27)) (justify right))
-    (property "Intersheetrefs" "${INTERSHEET_REFS}" (at 126.071 96.52 0)
-      (effects (font (size 1.27 1.27)) (justify right) hide)
-    )
-  )
   (global_label "BSPD_signal2" (shape input) (at 72.39 78.74 90) (fields_autoplaced)
     (effects (font (size 1.27 1.27)) (justify left))
@@
     )
   )
+  (global_label "CAN_RX" (shape input) (at 135.89 96.52 180) (fields_autoplaced)
+    (effects (font (size 1.27 1.27)) (justify right))
+    (property "Intersheetrefs" "${INTERSHEET_REFS}" (at 125.7686 96.52 0)
+      (effects (font (size 1.27 1.27)) (justify right) hide)
+    )
+  )
   (global_label "IMD_LED" (shape input) (at 135.89 78.74 180) (fields_autoplaced)
     (effects (font (size 1.27 1.27)) (justify right))
@@
     )
   )
+  (global_label "TSSI" (shape input) (at 107.95 114.3 90) (fields_autoplaced)
+    (effects (font (size 1.27 1.27)) (justify left))
+    (property "Intersheetrefs" "${INTERSHEET_REFS}" (at 107.95 107.3234 90)
+      (effects (font (size 1.27 1.27)) (justify left) hide)
+    )
+  )
   (global_label "USB_D+" (shape input) (at 240.03 123.19 180) (fields_autoplaced)
     (effects (font (size 1.27 1.27)) (justify right))
@@
     )
   )
-  (global_label "CAN_RX" (shape input) (at 135.89 99.06 180) (fields_autoplaced)
-    (effects (font (size 1.27 1.27)) (justify right))
-    (property "Intersheetrefs" "${INTERSHEET_REFS}" (at 125.7686 99.06 0)
-      (effects (font (size 1.27 1.27)) (justify right) hide)
+  (global_label "TSSI" (shape input) (at 53.34 182.88 0) (fields_autoplaced)
+    (effects (font (size 1.27 1.27)) (justify left))
+    (property "Intersheetrefs" "${INTERSHEET_REFS}" (at 60.3166 182.88 0)
+      (effects (font (size 1.27 1.27)) (justify left) hide)
     )
   )
@@
     )
   )
+  (symbol (lib_id "power:GND") (at 107.95 124.46 0) (unit 1)
+    (in_bom yes) (on_board yes) (dnp no) (fields_autoplaced)
+    (property "Reference" "#PWR047" (at 107.95 130.81 0)
+      (effects (font (size 1.27 1.27)) hide)
+    )
+    (property "Value" "GND" (at 107.95 129.54 0)
+      (effects (font (size 1.27 1.27)))
+    )
+    (property "Footprint" "" (at 107.95 124.46 0)
+      (effects (font (size 1.27 1.27)) hide)
+    )
+    (property "Datasheet" "" (at 107.95 124.46 0)
+      (effects (font (size 1.27 1.27)) hide)
+    )
+    (pin "1")
+    (instances
+      (project "rear-mcu"
+        (path "/df5b5f24-3d61-486a-be7e-cedc462763e6"
+          (reference "#PWR047") (unit 1)
+        )
+      )
+    )
+  )
   (symbol (lib_id "Switch:SW_SPST") (at 264.16 45.72 90) (unit 1)
     (in_bom yes) (on_board yes) (dnp no) (fields_autoplaced)
@@
     )
   )
-  (symbol (lib_id "power:+3.3V") (at 181.61 143.51 0) (unit 1)
+  (symbol (lib_id "power:+5V") (at 16.51 139.7 0) (unit 1)
     (in_bom yes) (on_board yes) (dnp no) (fields_autoplaced)
-    (property "Reference" "#PWR018" (at 181.61 147.32 0)
+    (property "Reference" "#PWR039" (at 16.51 143.51 0)
       (effects (font (size 1.27 1.27)) hide)
     )
-    (property "Value" "+3.3V" (at 181.61 138.43 0)
+    (property "Value" "+5V" (at 16.51 135.255 0)
       (effects (font (size 1.27 1.27)))
     )
-    (property "Footprint" "" (at 181.61 143.51 0)
+    (property "Footprint" "" (at 16.51 139.7 0)
       (effects (font (size 1.27 1.27)) hide)
     )
-    (property "Datasheet" "" (at 181.61 143.51 0)
+    (property "Datasheet" "" (at 16.51 139.7 0)
       (effects (font (size 1.27 1.27)) hide)
     )
@@
       (project "rear-mcu"
         (path "/df5b5f24-3d61-486a-be7e-cedc462763e6"
-          (reference "#PWR018") (unit 1)
+          (reference "#PWR039") (unit 1)
         )
       )
     )
   )
-  (symbol (lib_id "power:+5V") (at 16.51 139.7 0) (unit 1)
+  (symbol (lib_id "Device:R") (at 107.95 119.38 0) (unit 1)
     (in_bom yes) (on_board yes) (dnp no) (fields_autoplaced)
-    (property "Reference" "#PWR039" (at 16.51 143.51 0)
-      (effects (font (size 1.27 1.27)) hide)
+    (property "Reference" "R26" (at 110.49 118.11 0)
+      (effects (font (size 1.27 1.27)) (justify left))
     )
-    (property "Value" "+5V" (at 16.51 135.255 0)
-      (effects (font (size 1.27 1.27)))
+    (property "Value" "47k" (at 110.49 120.65 0)
+      (effects (font (size 1.27 1.27)) (justify left))
     )
-    (property "Footprint" "" (at 16.51 139.7 0)
+    (property "Footprint" "Resistor_SMD:R_0603_1608Metric" (at 106.172 119.38 90)
       (effects (font (size 1.27 1.27)) hide)
     )
-    (property "Datasheet" "" (at 16.51 139.7 0)
+    (property "Datasheet" "~" (at 107.95 119.38 0)
       (effects (font (size 1.27 1.27)) hide)
     )
     (pin "1")
+    (pin "2")
     (instances
       (project "rear-mcu"
         (path "/df5b5f24-3d61-486a-be7e-cedc462763e6"
-          (reference "#PWR039") (unit 1)
+          (reference "R26") (unit 1)
         )
       )
@@
         )
       )
+    )
+  )
+  (symbol (lib_id "power:+3.3V") (at 181.61 143.51 0) (unit 1)
+    (in_bom yes) (on_board yes) (dnp no) (fields_autoplaced)
+    (property "Reference" "#PWR018" (at 181.61 147.32 0)
+      (effects (font (size 1.27 1.27)) hide)
+    )
+    (property "Value" "+3.3V" (at 181.61 138.43 0)
+      (effects (font (size 1.27 1.27)))
+    )
+    (property "Footprint" "" (at 181.61 143.51 0)
+      (effects (font (size 1.27 1.27)) hide)
+    )
+    (property "Datasheet" "" (at 181.61 143.51 0)
+      (effects (font (size 1.27 1.27)) hide)
+    )
+    (pin "1")
+    (instances
+      (project "rear-mcu"
+        (path "/df5b5f24-3d61-486a-be7e-cedc462763e6"
+          (reference "#PWR018") (unit 1)
+        )
+      )

Commit message: v2025.5
Parts:
- removed R4: 47k, Resistor_SMD:R_0603_1608Metric, symbol Device:R
- removed R5: 100k, Resistor_SMD:R_0603_1608Metric, symbol Device:R
Connections:
- net BSPD_Check4: now reaches U1.17 (PA7)
- net BSPD_Check4: now also R1.2, R3.1
- removed net ADC_IN0: R1.2, R3.1, U1.10 (PA0)
- net BMS_signal renamed BMS_Fault
- net BSPD_signal renamed BSPD_Fault
- net Brake_signal1 renamed BSPD_signal4
- net Brake_signal2: no longer names the net of J1.9 (Pin_9)
- net IMD_signal renamed IMD_Fault
- no-connect marks 20 -> 19
Other:
- moved on the sheet: C11, C16, R14, R15, R22, R23, R26, U1, U2
