File: Charger_Mainboard/Charger_Mainboard.kicad_sch (KiCad schematic)
At the start: 34 parts, among them J10 Conn_02x10_Odd_Even, J11 Conn_01x02_Pin, J12 Conn_01x02_Pin, J13 Conn_01x02_Pin, J14 Conn_01x02_Pin, J15 Conn_01x02_Pin, J16 Conn_01x02_Pin, J17 Conn_01x02_Pin, J18 DB9_5, J19 DB9_5, J2 Conn_01x02_Pin, J3 Conn_01x02_Pin, J4 Conn_01x02_Pin, J5 Conn_01x02_Pin, J6 Conn_01x02_Pin, J7 Conn_01x02_Pin, J8 DB9_5, U1 AP2204K-ADJ, U2 TLV2371DBV, U3 AP2204K-ADJ

Commit message: charger mainboard v2025.6
Parts:
- removed J18, J19, J8: DB9_5, Connector_Dsub:DSUB-9_Female_Horizontal_P2.77x2.84mm_EdgePinOffset4.94mm_Housed_MountingHolesOffset7.48mm, symbol Connector:DE9_Plug_MountingHoles
- removed J2, J3, J4, J5, J6, J7: Conn_01x02_Pin, Connector_PinHeader_2.54mm:PinHeader_1x02_P2.54mm_Vertical, symbol Connector:Conn_01x02_Pin
- added C1: 1u, Capacitor_SMD:C_0603_1608Metric_Pad1.08x0.95mm_HandSolder, symbol Device:C_Small
- added J1, J2, J3, J4, J5, J6, J7: Conn_01x02, Connector_JST:JST_XH_B2B-XH-A_1x02_P2.50mm_Vertical, symbol Connector_Generic:Conn_01x02
- added J18, J21, J22, J8: Conn_01x04, Connector_JST:JST_XH_B4B-XH-A_1x04_P2.50mm_Vertical, symbol Connector_Generic:Conn_01x04
- added J19, J20, J23, J9: Conn_01x02_Pin, Connector_PinHeader_2.54mm:PinHeader_1x02_P2.54mm_Vertical, symbol Connector:Conn_01x02_Pin
- J10: footprint Connector_PinHeader_2.54mm:PinHeader_2x10_P2.54mm_Vertical -> Connector_PinSocket_2.54mm:PinSocket_2x10_P2.54mm_Vertical
Connections:
- net +12V: now also J9.1 (Pin_1); no longer U2.5 (V+)
- net +5V: now also J11.1 (Pin_1), U2.5 (V+), C1.1, J23.1 (Pin_1)
- net BMS_FAULT: now also J10.10 (Pin_10), J21.3 (Pin_3); no longer J10.9 (Pin_9)
- net BMS_LED: now also J10.9 (Pin_9), J22.2 (Pin_2); no longer J10.10 (Pin_10)
- net BMS_RST: now also J10.11 (Pin_11), J22.3 (Pin_3); no longer J10.12 (Pin_12)
- net GND: now also J10.15 (Pin_15), J10.19 (Pin_19), J10.2 (Pin_2), J10.6 (Pin_6), J10.8 (Pin_8), J16.1 (Pin_1), J16.2 (Pin_2), J17.1 (Pin_1), J17.2 (Pin_2), C1.2, J1.1 (Pin_1), J18.1 (Pin_1), J19.1 (Pin_1), J19.2 (Pin_2), J2.1 (Pin_1), J20.1 (Pin_1), J20.2 (Pin_2), J21.1 (Pin_1), J22.1 (Pin_1), J3.1 (Pin_1), J4.1 (Pin_1), J7.1 (Pin_1), J8.1 (Pin_1), J9.2 (Pin_2); no longer J10.1 (Pin_1), J10.16 (Pin_16), J10.20 (Pin_20), J10.5 (Pin_5), J10.7 (Pin_7), J11.1 (Pin_1), J12.1 (Pin_1), J13.1 (Pin_1), J15.1 (Pin_1)
- net IMD_FAULT: now also J10.13 (Pin_13), J21.4 (Pin_4); no longer J10.14 (Pin_14)
- net IMD_LED: now also J10.14 (Pin_14), J18.2 (Pin_2); no longer J10.13 (Pin_13)
- net IMD_RST: now also J10.12 (Pin_12), J18.3 (Pin_3); no longer J10.11 (Pin_11)
- net SDC_TO_SDBUTTON: now also J10.4 (Pin_4), J12.1 (Pin_1), J3.2 (Pin_2); no longer J10.3 (Pin_3)
- net VDC: now also J10.1 (Pin_1), J10.17 (Pin_17), J10.3 (Pin_3), J1.2 (Pin_2), J18.4 (Pin_4), J22.4 (Pin_4), J7.2 (Pin_2), J8.4 (Pin_4); no longer J10.2 (Pin_2), J10.4 (Pin_4), J14.1 (Pin_1), J14.2 (Pin_2)
- net charger_analog: now also J2.2 (Pin_2); no longer J15.2 (Pin_2)
- net BSPD_RST: now reaches J10.18 (Pin_18)
- net BSPD_RST: now also J8.3 (Pin_3)
- removed net FAN: J16.1 (Pin_1), J16.2 (Pin_2), J17.1 (Pin_1), J17.2 (Pin_2), R10.1
- new net BSPD_FAULT: J10.16 (Pin_16), J23.2 (Pin_2)
- new net BSPD_LED: J10.20 (Pin_20), J8.2 (Pin_2)
- new net FAN_PWM: J13.1 (Pin_1), J14.1 (Pin_1), J14.2 (Pin_2), J15.1 (Pin_1), J15.2 (Pin_2), J4.2 (Pin_2), J5.1 (Pin_1), J5.2 (Pin_2), J6.1 (Pin_1), J6.2 (Pin_2), R10.1
- new net SW_Fault: J10.7 (Pin_7)
- no-connect marks 14 -> 2
Other:
- note added: "12v backup"
- note added: "5v backup"
- note added: "BSPD Jumper"
- note added: "TSAL"
- note added: "VDC_in"
- note added: "X"
- note added: "from ACC box"
- note added: "to ACC box"
- moved on the sheet: C2, C3, C4, C5, J10, R6, R7, R8, R9, U1, U3

Commit message: add groung conn
Parts:
- added J24: Conn_01x02_Pin, Connector_PinHeader_2.54mm:PinHeader_1x02_P2.54mm_Vertical, symbol Connector:Conn_01x02_Pin
Connections:
- net GND: now also J24.1 (Pin_1), J24.2 (Pin_2)
Changed lines of the file:
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@@
+    )
+  )
+  (symbol (lib_id "Connector:Conn_01x02_Pin") (at 198.12 110.49 0) (mirror y) (unit 1)
+    (in_bom yes) (on_board yes) (dnp no) (fields_autoplaced)
+    (property "Reference" "J24" (at 197.485 105.41 0)
+      (effects (font (size 1.27 1.27)))
+    )
+    (property "Value" "Conn_01x02_Pin" (at 197.485 107.95 0)
+      (effects (font (size 1.27 1.27)) hide)
+    )
+    (property "Footprint" "Connector_PinHeader_2.54mm:PinHeader_1x02_P2.54mm_Vertical" (at 198.12 110.49 0)
+      (effects (font (size 1.27 1.27)) hide)
+    )
+    (property "Datasheet" "~" (at 198.12 110.49 0)
+      (effects (font (size 1.27 1.27)) hide)
+    )
+    (pin "1")
+    (pin "2")
+    (instances
+      (project "Charger_Mainboard"
+        (path "/2c4254d4-da70-461a-9652-3037a2f51e33"
+          (reference "J24") (unit 1)
+        )
+      )
     )
   )
@@
     )
   )
+  (symbol (lib_id "power:GND") (at 193.04 113.03 270) (unit 1)
+    (in_bom yes) (on_board yes) (dnp no) (fields_autoplaced)
+    (property "Reference" "#PWR052" (at 186.69 113.03 0)
+      (effects (font (size 1.27 1.27)) hide)
+    )
+    (property "Value" "GND" (at 189.23 113.03 90)
+      (effects (font (size 1.27 1.27)) (justify right))
+    )
+    (property "Footprint" "" (at 193.04 113.03 0)
+      (effects (font (size 1.27 1.27)) hide)
+    )
+    (property "Datasheet" "" (at 193.04 113.03 0)
+      (effects (font (size 1.27 1.27)) hide)
+    )
+    (pin "1")
+    (instances
+      (project "Charger_Mainboard"
+        (path "/2c4254d4-da70-461a-9652-3037a2f51e33"
+          (reference "#PWR052") (unit 1)
+        )
+      )
+    )
+  )
   (symbol (lib_id "power:+5V") (at 109.22 163.83 270) (unit 1)
     (in_bom yes) (on_board yes) (dnp no) (fields_autoplaced)
@@
         )
       )
+    )
+  )
+  (symbol (lib_id "power:GND") (at 193.04 110.49 270) (unit 1)
+    (in_bom yes) (on_board yes) (dnp no) (fields_autoplaced)
+    (property "Reference" "#PWR051" (at 186.69 110.49 0)
+      (effects (font (size 1.27 1.27)) hide)
+    )
+    (property "Value" "GND" (at 189.23 110.49 90)
+      (effects (font (size 1.27 1.27)) (justify right))
+    )
+    (property "Footprint" "" (at 193.04 110.49 0)
+      (effects (font (size 1.27 1.27)) hide)
+    )
+    (property "Datasheet" "" (at 193.04 110.49 0)
+      (effects (font (size 1.27 1.27)) hide)
+    )
+    (pin "1")
+    (instances
+      (project "Charger_Mainboard"
+        (path "/2c4254d4-da70-461a-9652-3037a2f51e33"
+          (reference "#PWR051") (unit 1)
+        )
+      )

Commit message: Charger v2026.1
Parts:
- removed J10: Conn_02x10_Odd_Even, Connector_PinSocket_2.54mm:PinSocket_2x10_P2.54mm_Vertical, symbol Connector_Generic:Conn_02x10_Odd_Even
- removed J11, J12, J13, J14, J15, J16, J17, J19, J20, J23, J24, J9: Conn_01x02_Pin, Connector_PinHeader_2.54mm:PinHeader_1x02_P2.54mm_Vertical, symbol Connector:Conn_01x02_Pin
- removed J6: Conn_01x02, Connector_JST:JST_XH_B2B-XH-A_1x02_P2.50mm_Vertical, symbol Connector_Generic:Conn_01x02
- removed R10: 100R, Resistor_SMD:R_0603_1608Metric, symbol Device:R_Small
- removed R11: 100k, Resistor_SMD:R_0603_1608Metric, symbol Device:R_Small
- removed U2: TLV2371DBV, Package_TO_SOT_SMD:SOT-23-5, symbol Amplifier_Operational:TLV2371DBV
- removed U3: AP2204K-ADJ, Package_TO_SOT_SMD:SOT-23-5, symbol Regulator_Linear:AP2204K-ADJ
- added C10, C9: 22u, Capacitor_SMD:C_0805_2012Metric, symbol Device:C_Small
- added C11: 1u, Capacitor_SMD:C_0603_1608Metric, symbol Device:C
- added C12: 10u, Capacitor_SMD:C_0805_2012Metric, symbol Device:C
- added C7: 100n, Capacitor_SMD:C_0603_1608Metric, symbol Device:C_Small
- added C8: 12p, Capacitor_SMD:C_0603_1608Metric, symbol Device:C_Small
- added D1: LED_Small, LED_SMD:LED_0805_2012Metric, symbol Device:LED_Small
- added H1, H2, H3, H4: MountingHole_Pad, MountingHole:MountingHole_4.3mm_M4_ISO7380_Pad, symbol Mechanical:MountingHole_Pad
- added J10: Conn_02x13_Odd_Even, Connector_PinSocket_2.54mm:PinSocket_2x13_P2.54mm_Vertical, symbol Connector_Generic:Conn_02x13_Odd_Even
- added L1: 15uH, Inductor_SMD:L_Coilcraft_XAL6060-XXX, symbol Device:L_Small
- added R1, R2: 0, Resistor_SMD:R_0603_1608Metric, symbol Device:R
- added R10: 100k, Resistor_SMD:R_0603_1608Metric, symbol Device:R
- added R11: 165k, Resistor_SMD:R_0603_1608Metric, symbol Device:R
- added R3: 301k, Resistor_SMD:R_0603_1608Metric, symbol Device:R_Small
- added R4: 100k, Resistor_SMD:R_0603_1608Metric, symbol Device:R_Small
- added R5: 10k, Resistor_SMD:R_0603_1608Metric, symbol Device:R_Small
- added TP1, TP2, TP3: TestPoint, TestPoint:TestPoint_THTPad_D1.5mm_Drill0.7mm, symbol Connector:TestPoint
- added U2: AS331KTR-G1, Package_TO_SOT_SMD:SOT-23-5, symbol Project_Lib:AS331KTR-G1
- added U3: AP63200WU, Package_TO_SOT_SMD:TSOT-23-6, symbol Regulator_Switching:AP63200WU
- added U4: AP2204K-ADJ, Package_TO_SOT_SMD:SOT-23-5, symbol Regulator_Linear:AP2204K-ADJ
- C2: footprint Capacitor_SMD:C_0603_1608Metric_Pad1.08x0.95mm_HandSolder -> Capacitor_SMD:C_0603_1608Metric
- C3, C5: footprint Capacitor_SMD:C_0805_2012Metric_Pad1.18x1.45mm_HandSolder -> Capacitor_SMD:C_0805_2012Metric
- C4: value 1u -> 10u; footprint Capacitor_SMD:C_0603_1608Metric_Pad1.08x0.95mm_HandSolder -> Capacitor_SMD:C_0805_2012Metric
- J1, J3, J4, J5: footprint Connector_JST:JST_XH_B2B-XH-A_1x02_P2.50mm_Vertical -> Connector_AMASS:AMASS_XT60-M_1x02_P7.20mm_Vertical
- R8: value 100k -> 534k
- R9: value 301k -> 30k1
Connections:
- net +5V: now also C11.1, TP2.1, U2.5, U4.1 (VIN), U4.3 (EN); no longer R14.1
- net BMS_FAULT: now also J10.12 (Pin_12)
- net BMS_LED: now also J10.9 (Pin_9), R2.1
- net BMS_RST: now also J10.11 (Pin_11), R1.2
- net BSPD_FAULT: now also J10.17 (Pin_17)
- net BSPD_LED: now also J10.20 (Pin_20), R2.2
- net BSPD_RST: now also J10.18 (Pin_18), R1.1
- net GND: now also J1.2 (Pin_2), R9.2, C10.2, C11.2, C12.2, C9.2, H1.1, H2.1, H3.1, H4.1, J10.1 (Pin_1), J10.19 (Pin_19), J10.21 (Pin_21), J10.7 (Pin_7), J10.8 (Pin_8), R10.1, R4.1, R5.1, U2.2, U3.4 (GND), U4.2 (GND); no longer J1.1 (Pin_1), J3.1 (Pin_1), J4.1 (Pin_1), R8.1
- net IMD_FAULT: now also J10.14 (Pin_14)
- net IMD_LED: now also J10.15 (Pin_15)
- net IMD_RST: now also J10.13 (Pin_13)
- net SDC_TO_SDBUTTON: now also J3.1 (Pin_1)
- net VDC: now also C5.1, J1.1 (Pin_1), U3.2 (EN), U3.3 (IN); no longer J1.2 (Pin_2)
- net charger_analog: now also D1.2 (A), U2.4
- net at R8.2: now also R9.1, C8.2, U3.1 (FB); no longer R9.2
- net at C6.1, R12.2, R13.1: now also U2.1 (-)
- net +12V renamed +15V
- net +15V: now also R8.1, C10.1, C8.1, C9.1, J10.23 (Pin_23), J10.24 (Pin_24), L1.2, TP1.1; no longer C5.1, R9.1
- net FAN_PWM renamed SDC_FROM_SDBUTTON
- net SDC_FROM_SDBUTTON: now also J4.1 (Pin_1), R3.2
- new net: R10.2, R11.2, U4.4 (ADJ)
- new net: R3.1, R4.2, U2.3 (+)
- new net: C7.1, L1.1, U3.5 (SW)
- new net: C7.2, U3.6 (BST)
- new net: D1.1 (K), R5.2
- new net +3V3: C12.1, R11.1, R14.1, TP3.1, U4.5 (VOUT)
- new net SDC_OUT: J10.10 (Pin_10)
- no-connect marks 2 -> 10
Other:
- note added: "2.5V"
- note added: "ACDC降成24V進主板 因風扇需24在電池箱中 因此直接給24，且不須FAN_PWM VDC=24V"
- note added: "LED button"
- note added: "SDC MCU"
- note added: "To Chroma"
- note added: "To/From ACC Box"
- note added: "normal 3.75V"
- note added: "從 button 回來"
- note added: "從SDC MCU 出來"
- note added: "為了斷電路板電源 防止按鈕復位後繼續運作"
- note added: "經 MS 的 SDC 會控制AIR"
- note added: "經 button"
- note added: "電源"
- note added: "電源 input"
- note removed: "12v backup"
- note removed: "5v backup"
- note removed: "BSPD Jumper"
- note removed: "VDC_in"
- note removed: "X"
- note removed: "from ACC box"
- note removed: "to ACC box"
- moved on the sheet: C1, C6, J1, J2, J21, J7, R12, R13, R14
