File: lv_mainboard/lv_mainboard.kicad_pcb (KiCad board)
At the start: 2 copper layers, 102 x 202 mm, 21 parts, among them J1 DE9_Plug, J15 Conn_02x10_Counter_Clockwise, J16 Conn_02x10_Counter_Clockwise, J17 Conn_02x10_Counter_Clockwise, J19 Conn_02x10_Counter_Clockwise, J2 DE9_Plug, J21 Conn_02x10_Counter_Clockwise, J3 DE9_Plug, J4 DE9_Plug, J5 DE9_Plug

Commit message: add layout
Parts:
- removed J16, J17, J19, J21: Conn_02x10_Counter_Clockwise, Connector_PinSocket_2.54mm:PinSocket_2x10_P2.54mm_Vertical
- added H1: MountingHole, MountingHole:MountingHole_4.3mm_M4_Pad, F.Cu at (161.0, 43.0)
- added H2: MountingHole, MountingHole:MountingHole_4.3mm_M4_Pad, F.Cu at (251.0, 43.0)
- added H3: MountingHole, MountingHole:MountingHole_4.3mm_M4_Pad, F.Cu at (161.0, 233.0)
- added H4: MountingHole, MountingHole:MountingHole_4.3mm_M4_Pad, F.Cu at (251.0, 233.0)
- added J13: Conn_02x10_Odd_Even, Connector_PinSocket_2.54mm:PinSocket_2x10_P2.54mm_Vertical, F.Cu at (182.2, 47.5)
- added J14: Conn_02x10_Odd_Even, Connector_PinSocket_2.54mm:PinSocket_2x10_P2.54mm_Vertical, F.Cu at (218.2, 168.5)
- added J6: Conn_02x10_Odd_Even, Connector_PinSocket_2.54mm:PinSocket_2x10_P2.54mm_Vertical, F.Cu at (184.1, 174.5)
- added J7: Conn_02x10_Odd_Even, Connector_PinSocket_2.54mm:PinSocket_2x10_P2.54mm_Vertical, F.Cu at (183.1, 112.5)
- added R1: 100R, Resistor_SMD:R_0603_1608Metric, F.Cu at (246.4, 163.2)
- added R2: 47R, Resistor_SMD:R_0603_1608Metric, F.Cu at (250.3, 161.2)
- added R3: 100R, Resistor_SMD:R_0603_1608Metric, F.Cu at (246.3, 168.0)
- added R4: 47R, Resistor_SMD:R_0603_1608Metric, F.Cu at (246.3, 172.8)
- added R5: 100R, Resistor_SMD:R_0603_1608Metric, F.Cu at (250.3, 170.8)
- added R6: 47R, Resistor_SMD:R_0603_1608Metric, F.Cu at (250.3, 166.0)
- added TP1: TestPoint, TestPoint:TestPoint_Keystone_5000-5004_Miniature, F.Cu at (190.0, 228.0)
- added TP10: TestPoint, TestPoint:TestPoint_Keystone_5000-5004_Miniature, F.Cu at (234.0, 225.0)
- added TP15: TestPoint, TestPoint:TestPoint_Keystone_5000-5004_Miniature, F.Cu at (169.0, 173.0)
- added TP16: TestPoint, TestPoint:TestPoint_Keystone_5000-5004_Miniature, F.Cu at (170.0, 86.0)
- added TP17: TestPoint, TestPoint:TestPoint_Keystone_5000-5004_Miniature, F.Cu at (170.0, 80.0)
- added TP18: TestPoint, TestPoint:TestPoint_Keystone_5000-5004_Miniature, F.Cu at (170.0, 74.0)
- added TP19: TestPoint, TestPoint:TestPoint_Keystone_5000-5004_Miniature, F.Cu at (170.0, 68.0)
- added TP2: TestPoint, TestPoint:TestPoint_Keystone_5000-5004_Miniature, F.Cu at (203.0, 228.0)
- added TP20: TestPoint, TestPoint:TestPoint_Keystone_5000-5004_Miniature, F.Cu at (170.0, 62.0)
- added TP21: TestPoint, TestPoint:TestPoint_Keystone_5000-5004_Miniature, F.Cu at (170.0, 56.0)
- added TP3: TestPoint, TestPoint:TestPoint_Keystone_5000-5004_Miniature, F.Cu at (172.0, 228.0)
- added TP4: TestPoint, TestPoint:TestPoint_Keystone_5000-5004_Miniature, F.Cu at (166.8, 145.8)
- added TP5: TestPoint, TestPoint:TestPoint_Keystone_5000-5004_Miniature, F.Cu at (166.8, 134.3)
- added TP6: TestPoint, TestPoint:TestPoint_Keystone_5000-5004_Miniature, F.Cu at (239.0, 225.0)
- added TP7: TestPoint, TestPoint:TestPoint_Keystone_5000-5004_Miniature, F.Cu at (229.0, 225.0)
- J1, J2, J3, J4, J5: footprint Connector_Dsub:DSUB-9_Female_Vertical_P2.77x2.84mm -> Connector_Dsub:DSUB-9_Female_Horizontal_P2.77x2.84mm_EdgePinOffset7.70mm_Housed_MountingHolesOffset9.12mm
- moved TP13 112.6 mm to (214.0, 225.0)
- moved TP9 75.7 mm to (169.0, 162.0)
- moved TP14 50.6 mm to (169.0, 180.0)
- moved TP11 29.0 mm to (219.0, 225.0)
- moved TP12 20.8 mm to (224.0, 225.0)
- moved J10 16.4 mm to (160.0, 143.0)
- moved J5 15.3 mm to (161.8, 113.0)
- moved J9 15.1 mm to (160.0, 131.5)
- moved J4 13.7 mm to (161.8, 76.1)
- moved J1 13.3 mm to (231.7, 233.2)
- moved J2 13.2 mm to (161.4, 174.4)
- moved J3 13.2 mm to (161.4, 210.5)
- moved J15 9.55 mm to (220.2, 102.5)
- moved J37 9.49 mm to (187.0, 233.0)
- moved J38 9.49 mm to (200.0, 233.0)
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Connections:
- net Net-(J8-Pin_2) renamed BSPD_IN
- J1 pad 1: unconnected-(J1-Pad1) -> +12V
- J1 pad 2: unconnected-(J1-Pad2) -> IMD_LED
- J1 pad 4: unconnected-(J1-Pad4) -> IMD_RST
- J1 pad 5: unconnected-(J1-Pad5) -> GND
- J1 pad 6: unconnected-(J1-Pad6) -> BSPD_LED
- J1 pad 7: unconnected-(J1-Pad7) -> BMS_LED
- J1 pad 8: unconnected-(J1-Pad8) -> BSPD_RST
- J1 pad 9: unconnected-(J1-Pad9) -> BMS_RST
- J10 pad 2: Net-(J10-Pin_2) -> Brake_init
- J2 pad 1: unconnected-(J2-Pad1) -> +24V
- J2 pad 2: unconnected-(J2-Pad2) -> CAN+
- J2 pad 5: unconnected-(J2-Pad5) -> GND
- J2 pad 6: unconnected-(J2-Pad6) -> CAN-
- J37 pad 2: Net-(J37-Pin_2) -> IMD_FAULT
- J38 pad 2: Net-(J38-Pin_2) -> BMS_FAULT
- J4 pad 1: unconnected-(J4-Pad1) -> FAN_PWM
- J4 pad 2: unconnected-(J4-Pad2) -> PT_signal
- J4 pad 3: unconnected-(J4-Pad3) -> USART1
- J4 pad 5: unconnected-(J4-Pad5) -> GND
- J4 pad 6: unconnected-(J4-Pad6) -> PUMP_PWM
- J4 pad 7: unconnected-(J4-Pad7) -> TIM1_CH1
- J4 pad 8: unconnected-(J4-Pad8) -> USART2
- J8 pad 1: GND -> SW_OUT
- J9 pad 2: Net-(J9-Pin_2) -> Current_init
- TP11 pad 1: Net-(J37-Pin_2) -> BSPD_RST
- TP12 pad 1: Net-(J38-Pin_2) -> IMD_RST
- TP13 pad 1: Net-(J9-Pin_2) -> BMS_RST
- TP14 pad 1: Net-(J10-Pin_2) -> CAN-
- TP9 pad 1: unconnected-(TP9-Pad1) -> SW_Fault
Routing:
- net CAN+: track 0.00 -> 243.1 mm
- net CAN-: track 0.00 -> 226.1 mm, vias 0 -> 3
- net VDC: track 0.00 -> 211.3 mm, vias 0 -> 2
- net BSPD_LED: track 0.00 -> 118.3 mm, vias 0 -> 2
- net BMS_LED: track 0.00 -> 111.3 mm, vias 0 -> 2
- net IMD_LED: track 0.00 -> 93.5 mm, vias 0 -> 2
- net Brake_Limit_Check_out: track 0.00 -> 90.0 mm
- net IMD_RST: track 0.00 -> 87.9 mm
- net Current_Limit_Check_out: track 0.00 -> 83.5 mm
- net BMS_FAULT: track 0.00 -> 80.5 mm, vias 0 -> 1
- net Simultaneous_brake&current: track 0.00 -> 78.8 mm
- net SW_Fault: track 0.00 -> 78.5 mm, vias 0 -> 1
- net BSPD_RST: track 0.00 -> 76.8 mm
- net BMS_RST: track 0.00 -> 72.5 mm
- net SW_OUT: track 0.00 -> 69.9 mm, vias 0 -> 1
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- added copper zone on B.Cu, net GND
- added copper zone on F.Cu, net GND
Other:
- outline, holes or cut-outs redrawn

Commit message: add mounting hole
Parts:
- removed R1, R3, R5: 100R, Resistor_SMD:R_0603_1608Metric
- removed R2, R4, R6: 47R, Resistor_SMD:R_0603_1608Metric
- removed TP14, TP15: TestPoint, TestPoint:TestPoint_Keystone_5000-5004_Miniature
- added H10: MountingHole_Pad, MountingHole:MountingHole_3.2mm_M3_Pad, F.Cu at (245.0, 82.0)
- added H11: MountingHole_Pad, MountingHole:MountingHole_3.2mm_M3_Pad, F.Cu at (245.0, 144.0)
- added H12: MountingHole_Pad, MountingHole:MountingHole_3.2mm_M3_Pad, F.Cu at (287.0, 144.0)
- added H13: MountingHole_Pad, MountingHole:MountingHole_3.2mm_M3_Pad, F.Cu at (237.0, 156.0)
- added H14: MountingHole_Pad, MountingHole:MountingHole_3.2mm_M3_Pad, F.Cu at (200.0, 156.0)
- added H15: MountingHole_Pad, MountingHole:MountingHole_3.2mm_M3_Pad, F.Cu at (200.0, 203.0)
- added H16: MountingHole_Pad, MountingHole:MountingHole_3.2mm_M3_Pad, F.Cu at (237.0, 203.0)
- added H17: MountingHole_Pad, MountingHole:MountingHole_3.2mm_M3_Pad, F.Cu at (198.0, 227.0)
- added H18: MountingHole_Pad, MountingHole:MountingHole_3.2mm_M3_Pad, F.Cu at (198.0, 289.0)
- added H19: MountingHole_Pad, MountingHole:MountingHole_3.2mm_M3_Pad, F.Cu at (235.0, 289.0)
- added H20: MountingHole_Pad, MountingHole:MountingHole_3.2mm_M3_Pad, F.Cu at (235.0, 227.0)
- added H21: MountingHole_Pad, MountingHole:MountingHole_3.2mm_M3_Pad, F.Cu at (283.0, 244.0)
- added H22: MountingHole_Pad, MountingHole:MountingHole_3.2mm_M3_Pad, F.Cu at (283.0, 286.0)
- added H23: MountingHole_Pad, MountingHole:MountingHole_3.2mm_M3_Pad, F.Cu at (261.0, 244.0)
- added H24: MountingHole_Pad, MountingHole:MountingHole_3.2mm_M3_Pad, F.Cu at (261.0, 286.0)
- added H5: MountingHole_Pad, MountingHole:MountingHole_3.2mm_M3_Pad, F.Cu at (225.0, 91.0)
- added H6: MountingHole_Pad, MountingHole:MountingHole_3.2mm_M3_Pad, F.Cu at (225.0, 133.0)
- added H7: MountingHole_Pad, MountingHole:MountingHole_3.2mm_M3_Pad, F.Cu at (203.0, 133.0)
- added H8: MountingHole_Pad, MountingHole:MountingHole_3.2mm_M3_Pad, F.Cu at (203.0, 91.0)
- added H9: MountingHole_Pad, MountingHole:MountingHole_3.2mm_M3_Pad, F.Cu at (287.0, 82.0)
- added J11: Conn_02x05_Counter_Clockwise, Connector_PinSocket_2.54mm:PinSocket_2x05_P2.54mm_Vertical, F.Cu at (287.6, 108.0)
- added J12: Conn_01x03, Connector_JST:JST_EH_B3B-EH-A_1x03_P2.50mm_Vertical, F.Cu at (235.5, 314.0)
- added TP24: TestPoint, TestPoint:TestPoint_Keystone_5000-5004_Miniature, F.Cu at (182.6, 244.7)
- added TP25: TestPoint, TestPoint:TestPoint_Keystone_5000-5004_Miniature, F.Cu at (182.6, 222.7)
- H1, H2, H3, H4: value MountingHole -> MountingHole_Pad
- moved H3 163.4 mm to (304.0, 312.0)
- moved TP9 153.7 mm to (214.0, 309.0)
- moved H4 108.9 mm to (176.0, 312.0)
- moved J15 108.8 mm to (293.0, 183.4), turned to 0 degrees
- moved J14 107.3 mm to (283.6, 253.6), turned to 0 degrees
- moved TP11 97.0 mm to (274.6, 304.5)
- moved J7 94.0 mm to (235.1, 190.9), turned to 180 degrees
- moved J1 89.2 mm to (272.3, 312.6)
- moved TP12 89.2 mm to (264.6, 304.5)
- moved TP13 89.2 mm to (254.6, 304.5)
- moved TP6 89.2 mm to (279.6, 304.5)
- moved TP7 89.2 mm to (269.6, 304.5)
- moved J6 88.5 mm to (235.6, 246.6), turned to 0 degrees
- moved J38 83.6 mm to (220.5, 314.0)
- moved TP10 83.5 mm to (259.6, 304.5)
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Connections:
- H1 pad 1: (no net) -> GND
- H2 pad 1: (no net) -> GND
- H3 pad 1: (no net) -> GND
- H4 pad 1: (no net) -> GND
- J1 pad 1: +12V -> BSPD_LED
- J1 pad 2: IMD_LED -> BMS_LED
- J1 pad 3: unconnected-(J1-Pad3) -> IMD_LED
- J1 pad 5: GND -> BSPD_RST
- J1 pad 6: BSPD_LED -> +12V
- J1 pad 7: BMS_LED -> unconnected-(J1-Pad7)
- J1 pad 8: BSPD_RST -> GND
- J14 pad 10: BSPD_signal1 -> Brake_Limit_Check_out
- J14 pad 12: BSPD_signal2 -> Current_Limit_Check_out
- J14 pad 14: BSPD_signal3 -> Simultaneous_brake&current
- J2 pad 3: unconnected-(J2-Pad3) -> CAN-
- J2 pad 4: unconnected-(J2-Pad4) -> CAN+
- J2 pad 5: GND -> CAN-
- J2 pad 6: CAN- -> BSE1
- J2 pad 8: unconnected-(J2-Pad8) -> GND
- J2 pad 9: unconnected-(J2-Pad9) -> BSE2
- J4 pad 2: PT_signal -> PUMP_PWM
- J4 pad 3: USART1 -> PT_signal
- J4 pad 4: unconnected-(J4-Pad4) -> TIM1_CH1
- J4 pad 5: GND -> USART1
- J4 pad 6: PUMP_PWM -> GND
- J4 pad 7: TIM1_CH1 -> unconnected-(J4-Pad7)
- J4 pad 8: USART2 -> unconnected-(J4-Pad8)
- J4 pad 9: unconnected-(J4-Pad9) -> USART2
- TP10 pad 1: BMS_LED -> BSPD_RST
- TP11 pad 1: BSPD_RST -> BMS_LED
Routing:
- net SW_Fault: track 78.5 -> 145.2 mm
- net Simultaneous_brake&current: track 78.8 -> 126.1 mm, vias 0 -> 4
- net BSPD_signal3: track 44.9 -> 0.00 mm, vias 1 -> 0
- net SW_OUT: track 69.9 -> 114.6 mm
- net BSPD_FAULT: track 62.5 -> 106.4 mm, vias 1 -> 4
- net CAN-: track 226.1 -> 266.1 mm, vias 3 -> 2
- net VDC: track 211.3 -> 244.4 mm
- net BSPD_signal2: track 30.3 -> 0.00 mm
- net BSPD_signal1: track 29.9 -> 0.00 mm, vias 2 -> 0
- net Current_Limit_Check_out: track 83.5 -> 109.7 mm, vias 0 -> 1
- net BMS_LED: track 111.3 -> 136.5 mm, vias 2 -> 0
- net USART2: track 33.2 -> 56.9 mm
- net CAN+: track 243.1 -> 266.1 mm, vias 0 -> 2
- net IMD_RST: track 87.9 -> 65.6 mm
- net BSPD_RST: track 76.8 -> 56.3 mm
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Other:
- board size 102 x 202 mm -> 140 x 250 mm

Commit message: v2025.5 finish schemetic
Parts:
- removed J37, J38: ~, Connector_JST:JST_EH_B2B-EH-A_1x02_P2.50mm_Vertical
- removed TP1, TP10, TP11, TP12, TP13, TP16, TP17, TP18, TP19, TP2, TP20, TP21, TP24, TP25, TP3, TP4, TP5, TP6, TP7, TP8, TP9: TestPoint, TestPoint:TestPoint_Keystone_5000-5004_Miniature
- added J16: Conn_01x04, Connector_JST:JST_XH_B4B-XH-A_1x04_P2.50mm_Vertical, F.Cu at (244.0, 311.0)
- added R1: R, Resistor_SMD:R_0603_1608Metric, F.Cu at (196.7, 226.0)
- added R2: R, Resistor_SMD:R_0603_1608Metric, F.Cu at (196.7, 228.5)
- H1, H2, H3, H4: footprint MountingHole:MountingHole_4.3mm_M4_Pad -> MountingHole:MountingHole_4.3mm_M4_ISO7380_Pad
- H10, H11, H12, H13, H14, H15, H16, H17, H18, H19, H20, H21, H22, H23, H24, H5, H6, H7, H8, H9: footprint MountingHole:MountingHole_3.2mm_M3_Pad -> MountingHole:MountingHole_3.2mm_M3_ISO7380_Pad
- J1: value DE9_Plug -> Conn_01x02; footprint Connector_Dsub:DSUB-9_Female_Horizontal_P2.77x2.84mm_EdgePinOffset7.70mm_Housed_MountingHolesOffset9.12mm -> Connector_JST:JST_XH_B2B-XH-A_1x02_P2.50mm_Vertical
- J10: value ~ -> PWR; footprint Connector_JST:JST_EH_B2B-EH-A_1x02_P2.50mm_Vertical -> Connector_AMASS:AMASS_XT60-M_1x02_P7.20mm_Vertical
- J12: value Conn_01x03 -> Conn_01x04; footprint Connector_JST:JST_EH_B3B-EH-A_1x03_P2.50mm_Vertical -> Connector_JST:JST_XH_B4B-XH-A_1x04_P2.50mm_Vertical
- J14: value Conn_02x10_Odd_Even -> Conn_01x04; footprint Connector_PinSocket_2.54mm:PinSocket_2x10_P2.54mm_Vertical -> Connector_JST:JST_XH_B4B-XH-A_1x04_P2.50mm_Vertical
- J15: value Conn_02x10_Counter_Clockwise -> Conn_01x04; footprint Connector_PinSocket_2.54mm:PinSocket_2x10_P2.54mm_Vertical -> Connector_JST:JST_XH_B4B-XH-A_1x04_P2.50mm_Vertical
- J2: value DE9_Plug -> Conn_02x10_Odd_Even; footprint Connector_Dsub:DSUB-9_Female_Horizontal_P2.77x2.84mm_EdgePinOffset7.70mm_Housed_MountingHolesOffset9.12mm -> Connector_PinSocket_2.54mm:PinSocket_2x10_P2.54mm_Vertical
- J3: value DE9_Plug -> Conn_01x03; footprint Connector_Dsub:DSUB-9_Female_Horizontal_P2.77x2.84mm_EdgePinOffset7.70mm_Housed_MountingHolesOffset9.12mm -> Connector_JST:JST_XH_B3B-XH-A_1x03_P2.50mm_Vertical
- J4: value DE9_Plug -> Conn_01x04; footprint Connector_Dsub:DSUB-9_Female_Horizontal_P2.77x2.84mm_EdgePinOffset7.70mm_Housed_MountingHolesOffset9.12mm -> Connector_JST:JST_XH_B4B-XH-A_1x04_P2.50mm_Vertical
- J5: value DE9_Plug -> Conn_01x05; footprint Connector_Dsub:DSUB-9_Female_Horizontal_P2.77x2.84mm_EdgePinOffset7.70mm_Housed_MountingHolesOffset9.12mm -> Connector_JST:JST_XH_B5B-XH-A_1x05_P2.50mm_Vertical
- J8: value ~ -> Conn_01x04; footprint Connector_JST:JST_EH_B2B-EH-A_1x02_P2.50mm_Vertical -> Connector_JST:JST_XH_B4B-XH-A_1x04_P2.50mm_Vertical
- J9: value ~ -> DE9_Plug_MountingHoles; footprint Connector_JST:JST_EH_B2B-EH-A_1x02_P2.50mm_Vertical -> Connector_Dsub:DSUB-9_Female_Horizontal_P2.77x2.84mm_EdgePinOffset7.70mm_Housed_MountingHolesOffset9.12mm
- moved J4 179.0 mm to (178.0, 291.0)
- moved J3 168.5 mm to (178.5, 114.5)
- moved J1 159.2 mm to (178.5, 184.0), turned to -90 degrees
- moved J15 145.9 mm to (178.5, 93.0), turned to -90 degrees
- moved J10 119.3 mm to (219.9, 311.0), turned to 0 degrees
- moved H18 104.6 mm to (302.5, 283.5)
- moved H22 98.6 mm to (195.5, 240.6), turned to 180 degrees
- moved H23 76.5 mm to (195.5, 283.6), turned to 180 degrees
- moved H14 72.2 mm to (243.5, 213.6)
- moved H17 70.1 mm to (239.5, 283.5)
- moved H11 70.1 mm to (249.5, 74.0), turned to -90 degrees
- moved H20 70.0 mm to (302.5, 245.5)
- moved H21 64.6 mm to (218.5, 240.6), turned to 180 degrees
- moved J6 60.2 mm to (282.4, 284.4), turned to -90 degrees
- moved H16 59.3 mm to (195.5, 160.6)
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Connections:
- J1 pad 1: BSPD_LED -> GND
- J1 pad 2: BMS_LED -> current_init
- J10 pad 1: GND -> SDC_OUT
- J10 pad 2: Brake_init -> GND
- J11 pad 1: P2 -> P2_BSPD
- J11 pad 2: P1 -> P1_DAQ
- J11 pad 3: P4 -> P4_SDCOUT
- J11 pad 4: P3 -> P3_SDCPCB
- J11 pad 5: P6 -> P6_sideboard
- J11 pad 6: P5 -> P5_MCU
- J12 pad 1: unconnected-(J12-Pin_1-Pad1) -> GND
- J12 pad 2: unconnected-(J12-Pin_2-Pad2) -> BSPD_LED
- J12 pad 3: unconnected-(J12-Pin_3-Pad3) -> BSPD_RST
- J13 pad 1: VDC -> P1_DAQ
- J13 pad 3: VDC -> P1_DAQ
- J13 pad 5: VDC -> P1_DAQ
- J14 pad 1: VDC -> GND
- J14 pad 2: SW_Fault -> BMS_LED
- J14 pad 3: VDC -> BMS_RST
- J14 pad 4: BMS_LED -> P6_sideboard
- J15 pad 1: unconnected-(J15-Pin_1-Pad1) -> GND
- J15 pad 2: unconnected-(J15-Pin_2-Pad2) -> P9
- J15 pad 3: unconnected-(J15-Pin_3-Pad3) -> P8
- J15 pad 4: unconnected-(J15-Pin_4-Pad4) -> P7
- J2 pad 1: +24V -> P5_MCU
- J2 pad 2: CAN+ -> SW_signal
- J2 pad 3: CAN- -> P5_MCU
- J2 pad 4: CAN+ -> BMS_Fault
- J2 pad 5: CAN- -> P5_MCU
- J2 pad 6: BSE1 -> IMD_Fault
- J2 pad 7: unconnected-(J2-Pad7) -> BSPD_signal4
- J2 pad 8: GND -> BSPD
- J2 pad 9: BSE2 -> unconnected-(J2-Pin_9-Pad9)
- J3 pad 1: unconnected-(J3-Pad1) -> GND
- J3 pad 2: unconnected-(J3-Pad2) -> FAN_PWR
- J3 pad 3: unconnected-(J3-Pad3) -> PUMP_PWR
- J4 pad 1: FAN_PWM -> GND
- J4 pad 2: PUMP_PWM -> TSSI
- J4 pad 3: PT_signal -> IMD_FAULT
- J4 pad 4: TIM1_CH1 -> BMS_FAULT
- J5 pad 1: unconnected-(J5-Pad1) -> GND
- J5 pad 2: unconnected-(J5-Pad2) -> USART1
- J5 pad 3: unconnected-(J5-Pad3) -> TIM1_CH1
- J5 pad 4: unconnected-(J5-Pad4) -> PT_signal
- J5 pad 5: unconnected-(J5-Pad5) -> USART2
- J6 pad 1: GND -> P3_SDCPCB
- J6 pad 10: BMS_LED -> BMS_FAULT
- J6 pad 11: IMD_RST -> BMS_RST
- J6 pad 12: BMS_RST -> IMD_RST
- J6 pad 13: IMD_LED -> IMD_FAULT
- J6 pad 14: IMD_FAULT -> IMD_LED
- J6 pad 15: BSPD_FAULT -> GND
- J6 pad 16: GND -> BSPD_FAULT
- J6 pad 17: BSPD_RST -> P4_SDCOUT
- J6 pad 18: BSPD_IN -> BSPD_RST
- J6 pad 19: BSPD_LED -> GND
- J6 pad 2: VDC -> GND
- J6 pad 20: GND -> BSPD_LED
- J6 pad 3: SW_OUT -> P3_SDCPCB
- J6 pad 4: VDC -> SDC_OUT
- J6 pad 5: GND -> unconnected-(J6-Pin_5-Pad5)
- J6 pad 6: unconnected-(J6-Pin_6-Pad6) -> GND
- J6 pad 7: GND -> SW_Fault
- J6 pad 8: SW_Fault -> GND
- J6 pad 9: BMS_FAULT -> BMS_LED
- J7 pad 1: VDC -> P2_BSPD
- J7 pad 10: Simultaneous_brake&current -> BSE_R_Fault
- J7 pad 11: Current_init -> unconnected-(J7-Pin_11-Pad11)
- J7 pad 12: Simultaneous_brake&current -> unconnected-(J7-Pin_12-Pad12)
- J7 pad 13: Current_init -> unconnected-(J7-Pin_13-Pad13)
- J7 pad 14: BSPD_FAULT -> BSPD_signal3
- J7 pad 15: GND -> unconnected-(J7-Pin_15-Pad15)
- J7 pad 16: BSPD_FAULT -> BSPD_signal4
- J7 pad 17: GND -> unconnected-(J7-Pin_17-Pad17)
- J7 pad 18: GND -> BSPD
- J7 pad 19: GND -> current_init
- J7 pad 2: Brake_Limit_Check_out -> BSE_L_init
- J7 pad 20: GND -> BSPD
- J7 pad 3: VDC -> P2_BSPD
- J7 pad 4: Brake_Limit_Check_out -> BSE_R_init
- J7 pad 5: VDC -> unconnected-(J7-Pin_5-Pad5)
- J7 pad 6: Current_Limit_Check_out -> BSE_L_Fault
- J7 pad 7: Brake_init -> unconnected-(J7-Pin_7-Pad7)
- J7 pad 8: Current_Limit_Check_out -> unconnected-(J7-Pin_8-Pad8)
- J7 pad 9: Brake_init -> unconnected-(J7-Pin_9-Pad9)
- J8 pad 1: SW_OUT -> GND
- J8 pad 2: BSPD_IN -> TSAL
- J9 pad 1: GND -> BSE_L_init
- J9 pad 2: Current_init -> CAN-
Routing:
- net VDC: track 244.4 -> 0.00 mm, vias 2 -> 0
- net SW_Fault: track 145.2 -> 0.00 mm, vias 1 -> 0
- net BMS_LED: track 136.5 -> 0.00 mm
- net Simultaneous_brake&current: track 126.1 -> 0.00 mm, vias 4 -> 0
- net SW_OUT: track 114.6 -> 0.00 mm, vias 1 -> 0
- net Current_Limit_Check_out: track 109.7 -> 0.00 mm, vias 1 -> 0
- net BSPD_LED: track 109.5 -> 0.00 mm, vias 2 -> 0
- net BSPD_FAULT: track 106.4 -> 0.00 mm, vias 4 -> 0
- net IMD_LED: track 100.8 -> 0.00 mm, vias 3 -> 0
- net Brake_Limit_Check_out: track 95.3 -> 0.00 mm, vias 3 -> 0
- net CAN+: track 266.1 -> 176.4 mm, vias 2 -> 0
- net CAN-: track 266.1 -> 177.2 mm, vias 2 -> 0
- net BMS_RST: track 74.6 -> 0.00 mm
- net BMS_FAULT: track 73.7 -> 0.48 mm, vias 1 -> 0
- net TIM1_CH1: track 72.4 -> 0.21 mm
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Other:
- board text added: "-"
- board text added: "BSPD"
- board text added: "DAQ"
- board text added: "Fuse Box"
- board text added: "SDC"
- board text added: "rear MCU"

Commit message: finish layout
Parts:
- added C1: 1u, Resistor_SMD:R_0603_1608Metric, F.Cu at (298.9, 99.8)
- added C2: 10u, Resistor_SMD:R_0805_2012Metric, F.Cu at (304.9, 96.0)
- added C3: 1u, Resistor_SMD:R_0603_1608Metric, F.Cu at (299.0, 87.5)
- added C4: 10u, Resistor_SMD:R_0805_2012Metric, F.Cu at (305.0, 83.0)
- added C5: 1u, Capacitor_SMD:C_0603_1608Metric_Pad1.08x0.95mm_HandSolder, F.Cu at (299.0, 111.6)
- added C6: 10u, Capacitor_SMD:C_0805_2012Metric_Pad1.18x1.45mm_HandSolder, F.Cu at (305.5, 108.0)
- added J12: Conn_01x04, Connector_JST:JST_XH_B4B-XH-A_1x04_P2.50mm_Vertical, F.Cu at (262.0, 301.5)
- added J14: Conn_01x04, Connector_JST:JST_XH_B4B-XH-A_1x04_P2.50mm_Vertical, F.Cu at (280.0, 301.5)
- added J16: Conn_01x04, Connector_JST:JST_XH_B4B-XH-A_1x04_P2.50mm_Vertical, F.Cu at (244.0, 301.5)
- added J17: Conn_01x04, Connector_JST:JST_XH_B4B-XH-A_1x04_P2.50mm_Vertical, F.Cu at (304.5, 130.0)
- added R3: 100k, Resistor_SMD:R_0603_1608Metric, F.Cu at (303.1, 103.0)
- added R4: 301k, Resistor_SMD:R_0603_1608Metric, F.Cu at (306.9, 99.7)
- added R5: 100k, Resistor_SMD:R_0603_1608Metric, F.Cu at (303.2, 90.5)
- added R6: 165k, Resistor_SMD:R_0603_1608Metric, F.Cu at (307.0, 86.8)
- added R7: 100k, Resistor_SMD:R_0603_1608Metric, F.Cu at (303.7, 115.5)
- added R8: 866k, Resistor_SMD:R_0603_1608Metric, F.Cu at (307.5, 111.7)
- added TP1: TestPoint, TestPoint:TestPoint_THTPad_D1.5mm_Drill0.7mm, F.Cu at (299.5, 125.0)
- added TP2: TestPoint, TestPoint:TestPoint_THTPad_D1.5mm_Drill0.7mm, F.Cu at (299.5, 121.0)
- added TP3: TestPoint, TestPoint:TestPoint_THTPad_D1.5mm_Drill0.7mm, F.Cu at (299.5, 129.0)
- added U1: AP2204K-ADJ, Package_TO_SOT_SMD:SOT-23-5, F.Cu at (302.9, 99.5)
- added U2: AP2204K-ADJ, Package_TO_SOT_SMD:SOT-23-5, F.Cu at (303.0, 87.0)
- added U3: AP2204K-ADJ, Package_TO_SOT_SMD:SOT-23-5, F.Cu at (303.4, 111.5)
- added kibuzzard-682D880A: G***, kibuzzard-682D880A, F.Cu at (308.5, 94.5)
- added kibuzzard-682D8819: G***, kibuzzard-682D8819, F.Cu at (297.5, 76.0)
- added kibuzzard-682D8830: G***, kibuzzard-682D8830, F.Cu at (308.5, 107.5)
- added kibuzzard-682D8907: G***, kibuzzard-682D8907, F.Cu at (309.0, 127.5)
- added kibuzzard-682D8919: G***, kibuzzard-682D8919, F.Cu at (309.0, 125.0)
- added kibuzzard-682D8927: G***, kibuzzard-682D8927, F.Cu at (309.0, 122.5)
- added kibuzzard-682D8AF9: G***, kibuzzard-682D8AF9, F.Cu at (284.0, 316.5)
- added kibuzzard-682D8B11: G***, kibuzzard-682D8B11, F.Cu at (265.5, 316.5)
- added kibuzzard-682D8B7A: G***, kibuzzard-682D8B7A, F.Cu at (248.0, 316.5)
- added kibuzzard-682D8C28: G***, kibuzzard-682D8C28, F.Cu at (294.5, 306.5)
- added kibuzzard-682D8E18: G***, kibuzzard-682D8E18, F.Cu at (226.0, 75.0)
- R1, R2: moved to B.Cu
- moved J15 43.4 mm to (217.5, 74.0), turned to 180 degrees
- moved R2 33.6 mm to (201.0, 195.2), turned to -90 degrees
- moved J3 23.0 mm to (178.0, 91.5)
- moved J5 22.5 mm to (178.0, 112.5)
- moved R1 19.0 mm to (201.0, 207.5), turned to 90 degrees
- moved J1 11.3 mm to (178.5, 172.8)
- moved J10 6.00 mm to (213.9, 311.0), turned to 180 degrees
Connections:
- J11 pad 3: P4_SDCOUT -> P4_RGB
- J15 pad 2: P9 -> P7
- J15 pad 3: P8 -> P9
- J15 pad 4: P7 -> P8
- J2 pad 4: BMS_Fault -> BMS_FAULT
- J2 pad 6: IMD_Fault -> IMD_FAULT
- J4 pad 2: TSSI -> TSAL
- J4 pad 3: IMD_FAULT -> BMS_FAULT
- J4 pad 4: BMS_FAULT -> IMD_FAULT
- J6 pad 16: BSPD_FAULT -> BSPD
- J6 pad 17: P4_SDCOUT -> P3_SDCPCB
- J9 pad 9: +3.3V -> +3V3
Routing:
- net +3V3: track 0.00 -> 323.5 mm, vias 0 -> 2
- net P6_sideboard: track 0.00 -> 306.6 mm, vias 0 -> 2
- net P5_MCU: track 0.04 -> 298.7 mm
- net P3_SDCPCB: track 0.00 -> 227.9 mm, vias 0 -> 2
- net BSPD: track 0.42 -> 191.1 mm, vias 0 -> 2
- net BMS_FAULT: track 0.48 -> 144.5 mm, vias 0 -> 2
- net IMD_FAULT: track 0.00 -> 144.0 mm, vias 0 -> 2
- net P2_BSPD: track 0.00 -> 143.2 mm
- net BSPD_signal4: track 0.00 -> 98.2 mm
- net SDC_OUT: track 0.00 -> 89.1 mm
- net BSPD_signal3: track 0.69 -> 88.9 mm, vias 0 -> 1
- net BSE_R_Fault: track 0.64 -> 85.7 mm, vias 0 -> 1
- net BSE_L_Fault: track 0.10 -> 81.5 mm, vias 0 -> 1
- net P7: track 0.00 -> 70.2 mm
- net P1_DAQ: track 0.30 -> 65.3 mm
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Other:
- board text added: "GND LED RST VDD"
- board text added: "GND TASL BMS_F IMD_F"
- board text added: "GND TASL TSSI 24V"
- board text added: "GND U1 T1 P1 U2"
- board text added: "GND pump fan"
- board text added: "PWM"
- board text added: "current_in"
- board text added: "from ACC Box"
- board text added: "from HV Box"
- board text added: "to Mainhoop Light"

Commit message: v2025.6, add vdd to accbox
Parts:
- added G***: LOGO, logo:galaxy_logo_10mm, F.Cu at (307.2, 213.0)
- added G***: LOGO, logo:fire_shark_4mm, F.Cu at (307.0, 203.5)
- added G***: LOGO, logo:nckufs_logo_10mm, F.Cu at (307.0, 187.5)
- added J18: Conn_01x02, Connector_JST:JST_XH_B2B-XH-A_1x02_P2.50mm_Vertical, F.Cu at (191.8, 311.0)
- added J19: PWR, Connector_AMASS:AMASS_XT60-M_1x02_P7.20mm_Vertical, F.Cu at (215.9, 74.5)
- J15: value Conn_01x04 -> PWR; footprint Connector_JST:JST_XH_B4B-XH-A_1x04_P2.50mm_Vertical -> Connector_AMASS:AMASS_XT60-M_1x02_P7.20mm_Vertical
- moved J15 24.1 mm to (193.4, 74.5), turned to 0 degrees
- moved kibuzzard-682D8E18 10.6 mm to (236.5, 76.5)
Connections:
- J11 pad 8: P7 -> P7_ACC
- J15 pad 1: GND -> P8
- J15 pad 2: P7 -> GND
Routing:
- net P7_ACC: track 0.00 -> 340.4 mm
- net P7: track 70.2 -> 0.00 mm
- net P8: track 57.5 -> 66.9 mm, vias 0 -> 1
- net GND: track 0.00 -> 9.35 mm, vias 0 -> 2
- net +3V3: track 323.5 -> 321.5 mm
- net P9: track 49.5 -> 50.5 mm, vias 0 -> 1
Other:
- board text added: "lv mainboard v2025.6"
- board text added: "to ACC Box"
