File: control-board/control-board.kicad_sch (KiCad schematic)
At the start: 97 parts, among them J1 Conn_01x03, J10 DIN-4, J11 DIN-4, J12 Conn_01x03, J13 Conn_01x03, J14 Conn_01x02, J15 Conn_01x03, J16 Conn_01x02, J17 Conn_01x02, J18 Conn_01x02, J2 GPS_ANT, J3 LORA_ANT, J4 DIN-4, J5 DIN-4, J6 USB_C_Receptacle_USB2.0_16P, J7 Conn_01x03, J8 DIN-4, J9 DIN-4, Q1 2N7002, Q2 2N7002, SW1 SW_SPST, U1 STM32H743VITx, U2 NEO-XM, U3 TCAN1462VDRQ1, U4 AMS1117-3.3, U6 AMS1117-3.3, U7 TCAN1462VDRQ1, Y1 8M, Y2 32.768k

Commit message: feat: update schematic & adc
Parts:
- added R7: 150R, Resistor_SMD:R_0603_1608Metric, symbol Device:R_Small
Connections:
- net ADC_BPPS: now also J10.3; no longer J10.2
- net ADC_STEER: now also J10.2, R7.1; no longer J10.3
- net GND: now also R7.2
Other:
- note added: "ADC"
- note added: "Additional"
- note added: "Buzzer"
- note added: "CAN1(General)"
- note added: "CAN2(Inverter)"
- note added: "Fault signal"
- note added: "GPS"
- note added: "LoRA"
- note added: "M8_connector"
- note added: "MCU-stm32h7"
- note added: "Power & TP"
- note added: "ST-link"
- note added: "USB"
- moved on the sheet: BZ1, C1, C10, C11, C12, C13, C14, C15, C16, C17, C18, C2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
