File: lvbms/lvbms.kicad_sch (KiCad schematic)
At the start: 110 parts, among them J1 Conn_T1, J2 Conn_T2, J3 Conn_PWR, J4 Conn_CAN, J5 Conn_WAKE, J6 Conn_OLED, J7 PROG, J8 USB_C_Receptacle_USB2.0_16P, Q1 2N7002, Q2 DMN6040SK3, Q3 DMN6040SK3, Q4 2N7002, Q5 DXT5551P5, U1 BQ76942PFBR, U2 SN65HVD256D, U3 STM32F103C8Tx, Y1 8M, Y2 32.768k

Commit message: feat: LV BMS layout
Parts:
- added H1, H2, H3, H4: MountingHole, MountingHole:MountingHole_3.2mm_M3_DIN965, symbol Mechanical:MountingHole
- added J10, J9: Conn_02x08_Counter_Clockwise, Connector_PinHeader_2.54mm:PinHeader_2x08_P2.54mm_Vertical_SMD, symbol Connector_Generic:Conn_02x08_Counter_Clockwise
- J3: footprint Connector_JST:JST_XH_B2B-XH-A_1x02_P2.50mm_Vertical -> Connector_AMASS:AMASS_XT60-M_1x02_P7.20mm_Vertical
- U1: footprint BQ76942PFBR:QFP50P900X900X120-48N -> Package_QFP:TQFP-48_7x7mm_P0.5mm
Connections:
- net -VDC: now also J3.1 (Pin_1); no longer J3.2 (Pin_2)
- net CELL_A1: now also J10.10 (Pin_10), J10.11 (Pin_11), J10.12 (Pin_12), J10.9 (Pin_9)
- net CELL_A2: now also J10.5 (Pin_5), J10.6 (Pin_6), J10.7 (Pin_7), J10.8 (Pin_8)
- net CELL_A3: now also J10.1 (Pin_1), J10.2 (Pin_2), J10.3 (Pin_3), J10.4 (Pin_4)
- net CELL_A4: now also J9.13 (Pin_13), J9.14 (Pin_14), J9.15 (Pin_15), J9.16 (Pin_16)
- net CELL_A5: now also J9.10 (Pin_10), J9.11 (Pin_11), J9.12 (Pin_12), J9.9 (Pin_9)
- net CELL_A6: now also J9.5 (Pin_5), J9.6 (Pin_6), J9.7 (Pin_7), J9.8 (Pin_8)
- net CELL_A7: now also J9.1 (Pin_1), J9.2 (Pin_2), J9.3 (Pin_3), J9.4 (Pin_4)
- net GND: now also J10.13 (Pin_13), J10.14 (Pin_14), J10.15 (Pin_15), J10.16 (Pin_16)
- net at C10.2, C16.1, Q3.3 (S)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: now also J3.2 (Pin_2); no longer J3.1 (Pin_1)

Commit message: feat: README version of LVBMS
Other:
- moved on the sheet: J10, J9
