File: bms-slave-panel/bms-slave-panel.kicad_pcb (KiCad board)
At the start: 2 copper layers, 269 x 80 mm, 65 parts, among them J1 Conn_02x10_Odd_Even, J2 Conn_02x10_Odd_Even, J3 Conn_02x10_Odd_Even, J4 Conn_02x10_Odd_Even

Commit message: fix: change direction of pinheader
Parts:
- moved R10 58.6 mm to (233.0, 55.0)
- moved R11 58.6 mm to (216.0, 55.0)
- moved R12 58.6 mm to (199.5, 55.0)
- moved R13 58.6 mm to (183.0, 55.0)
- moved R14 58.6 mm to (167.5, 55.0)
- moved R9 58.6 mm to (249.0, 55.0)
- moved R8 58.5 mm to (264.0, 55.0)
- moved TH10 53.6 mm to (232.9, 57.5)
- moved TH11 53.6 mm to (216.1, 57.5)
- moved TH12 53.6 mm to (199.5, 57.5)
- moved TH13 53.6 mm to (183.0, 57.5)
- moved TH14 53.6 mm to (167.5, 57.5)
- moved TH9 53.6 mm to (248.9, 57.5)
- moved TH8 53.5 mm to (264.0, 57.5)
- moved J4 28.7 mm to (277.0, 71.0), turned to 0 degrees
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Routing:
- net /B01: track 46.3 -> 8.47 mm, vias 1 -> 0
- net /B03: track 65.8 -> 33.7 mm, vias 1 -> 0
- net /B05: track 78.2 -> 49.1 mm, vias 1 -> 0
- net /B02: track 10.0 -> 36.3 mm, vias 0 -> 1
- net /B07: track 88.3 -> 68.7 mm, vias 1 -> 0
- net /B06: track 50.9 -> 68.0 mm, vias 0 -> 1
- net /B09: track 102.9 -> 87.7 mm, vias 1 -> 0
- net /B08: track 69.1 -> 83.5 mm, vias 0 -> 1
- net /NTCB03: track 46.0 -> 56.2 mm
- net 5VB: track 129.8 -> 121.1 mm
- net /B10: track 88.3 -> 96.9 mm, vias 0 -> 1
- net /NTCB05: track 80.9 -> 88.5 mm
- net /NTCB01: track 15.4 -> 22.0 mm
- net /NTCB07: track 113.0 -> 118.5 mm
- net /B04: track 36.1 -> 41.1 mm, vias 0 -> 1
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
Commit message: fix: panel layout
Routing:
- net /A10: track 0.00 -> 85.7 mm, vias 0 -> 1
- net /A09: track 69.8 -> 71.2 mm
- net /A14: track 66.6 -> 67.8 mm
- net /B13: track 130.9 -> 132.1 mm
- net /A01: track 288.8 -> 289.9 mm
- net /A04: track 127.4 -> 128.4 mm
- net /A05: track 104.5 -> 105.4 mm
- net /A12: track 75.0 -> 75.8 mm
- net /B05: track 49.1 -> 49.8 mm
- net /A03: track 120.4 -> 119.8 mm
- net /B03: track 33.7 -> 34.2 mm

Commit message: fix: remove filled zone
Routing:
- net GND: track 0.00 -> 135.1 mm
- net GND1: track 0.00 -> 130.0 mm
- removed copper zone on B.Cu, net GND
- removed copper zone on F.Cu, net GND
- removed copper zone on B.Cu, net GND1
- removed copper zone on F.Cu, net GND1
