File: TSAL/TSAL.kicad_sch (KiCad schematic)
At the start: 118 parts, among them IC3 LTC6995IS6-2#TRMPBF, IC4 LTC6995IS6-2#TRMPBF, J1 Conn_SDC, J2 Conn_TSAL, J3 Conn_AIR, J4 Conn_01x02, J5 Conn_VI, J6 Conn_PRE, J7 Conn_HV, J8 Conn_control, K1 G2RL-2, Q1 2N7002, Q2 2N7002, Q3 2N7002, Q4 2N7002, Q5 DN2470K4, U1 AMC1351, U10 TLV7041DBV, U2 TLV7041DBV, U3 AS331KTR-G1, U4 AS331KTR-G1, U5 74LVC1G08, U6 AP2205-W5-7, U7 AP2205-W5-7, U8 AMC1351, U9 AP2204K-ADJ

Commit message: fix: replace NMOS and div resistors
Parts:
- removed R10, R11, R14, R16, R18, R19, R39, R46, R47, R48, R8, R9: 1M, Resistor_SMD:R_0603_1608Metric, symbol Device:R
- removed RV3: 1k, Potentiometer_THT:Potentiometer_Bourns_3296W_Vertical, symbol Device:R_Potentiometer_Small
- removed U10: TLV7041DBV, Package_TO_SOT_SMD:SOT-23-5, symbol Comparator:TLV7041DBV
- added R10, R11, R14, R16, R18, R19, R39, R46, R47, R48, R51, R52, R53, R54, R55, R56, R57, R58, R59, R60, R61, R62, R8, R9: 500k, Resistor_SMD:R_0603_1608Metric, symbol Device:R_Small
- added R63: 1k, Resistor_SMD:R_0805_2012Metric, symbol Device:R
- added U10: AS331KTR-G1, Package_TO_SOT_SMD:SOT-23-5, symbol Project_Lib:AS331KTR-G1
- Q5: value DN2470K4 -> IXTP01N100D; footprint Package_TO_SOT_SMD:TO-252-2 -> Package_TO_SOT_THT:TO-220-3_Vertical
Connections:
- net +5VA: now also U10.5
- net BATT+: now also R55.1
- net GND1: now also U10.2
- net HV+: now also R39.1, R8.1
- net at Q5.3 (S), R49.1, R50.1: now also R63.1
- net at J5.1 (Pin_1), Q5.1 (G), R49.2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: now also R63.2
- net at C8.1, R12.2, U1.2 (+): now also R19.2
- net at C4.1, U8.2 (+): now also U10.4
- net at R15.2: now also R54.2, U10.3 (+)
- net at R17.1: now also R62.2, U10.1 (-)
- new net: R39.2, R46.1
- new net: R46.2, R47.1
- new net: R16.2, R18.1
- new net: R18.2, R19.1
- new net: R51.2, R52.1
- new net: R52.2, R53.1
- new net: R57.2, R58.1
- new net: R58.2, R59.1
- new net: R10.2, R11.1
- new net: R11.2, R14.1
- new net: R14.2, R16.1
- new net: R55.2, R56.1
- new net: R56.2, R57.1
- new net: R8.2, R9.1
- new net: R10.1, R9.2
- new net: R60.2, R61.1
- new net: R61.2, R62.1
- new net: R48.2, R51.1
- new net: R53.2, R54.1
- new net: R59.2, R60.1
- new net: R47.2, R48.1
Other:
- moved on the sheet: C1, C10, C16, C17, C2, C20, C21, C22, C23, C24, C25, C26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
