File: bms-slave/BQ79616_BMS_14Ch.kicad_sch (KiCad schematic)
At the start: 158 parts, among them J2 Conn_02x12_Odd_Even, J4 BMS_A_OUT, J5 BMS_A_IN, Q1 DXT5551P5, Q10 DMN2024UQ, Q11 DMN2024UQ, Q12 DMN2024UQ, Q13 DMN2024UQ, Q14 DMN2024UQ, Q15 DMN2024UQ, Q2 DMN2024UQ, Q3 DMN2024UQ, Q4 DMN2024UQ, Q5 DMN2024UQ, Q6 DMN2024UQ, Q7 DMN2024UQ, Q8 DMN2024UQ, Q9 DMN2024UQ

Commit message: fix: fuse & tvs package
Parts:
- D1, D10, D11, D12, D13, D14, D2, D3, D4, D5, D6, D7, D8, D9: footprint Fuse:Fuse_2512_6332Metric_Pad1.52x3.35mm_HandSolder -> Diode_SMD:D_SMB
- F1, F10, F11, F12, F13, F14, F15, F2, F3, F4, F5, F6, F7, F8, F9: footprint Fuse:Fuse_0805_2012Metric -> Fuse:Fuse_2512_6332Metric_Pad1.52x3.35mm_HandSolder
Changed lines of the file:
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@@
 			)
 		)
-		(property "Footprint" "Fuse:Fuse_0805_2012Metric"
+		(property "Footprint" "Fuse:Fuse_2512_6332Metric_Pad1.52x3.35mm_HandSolder"
 			(at 36.83 335.28 0)
 			(effects
@@
 			)
 		)
-		(property "Footprint" "Fuse:Fuse_2512_6332Metric_Pad1.52x3.35mm_HandSolder"
+		(property "Footprint" "Diode_SMD:D_SMB"
 			(at 43.815 248.285 0)
 			(effects
@@
 			)
 		)
-		(property "Footprint" "Fuse:Fuse_0805_2012Metric"
+		(property "Footprint" "Fuse:Fuse_2512_6332Metric_Pad1.52x3.35mm_HandSolder"
 			(at 36.83 201.93 0)
 			(effects
@@
 			)
 		)
-		(property "Footprint" "Fuse:Fuse_0805_2012Metric"
+		(property "Footprint" "Fuse:Fuse_2512_6332Metric_Pad1.52x3.35mm_HandSolder"
 			(at 36.83 297.18 0)
 			(effects
@@
 			)
 		)
-		(property "Footprint" "Fuse:Fuse_2512_6332Metric_Pad1.52x3.35mm_HandSolder"
+		(property "Footprint" "Diode_SMD:D_SMB"
 			(at 43.815 286.385 0)
 			(effects
@@
 			)
 		)
-		(property "Footprint" "Fuse:Fuse_2512_6332Metric_Pad1.52x3.35mm_HandSolder"
+		(property "Footprint" "Diode_SMD:D_SMB"
 			(at 43.815 95.885 0)
 			(effects
@@
 			)
 		)
-		(property "Footprint" "Fuse:Fuse_2512_6332Metric_Pad1.52x3.35mm_HandSolder"
+		(property "Footprint" "Diode_SMD:D_SMB"
 			(at 43.815 210.185 0)
 			(effects
@@
 			)
 		)
-		(property "Footprint" "Fuse:Fuse_0805_2012Metric"
+		(property "Footprint" "Fuse:Fuse_2512_6332Metric_Pad1.52x3.35mm_HandSolder"
 			(at 36.83 240.03 0)
 			(effects
@@
 			)
 		)
-		(property "Footprint" "Fuse:Fuse_2512_6332Metric_Pad1.52x3.35mm_HandSolder"
+		(property "Footprint" "Diode_SMD:D_SMB"
 			(at 43.815 343.535 0)
 			(effects
@@
 			)
 		)
-		(property "Footprint" "Fuse:Fuse_2512_6332Metric_Pad1.52x3.35mm_HandSolder"
+		(property "Footprint" "Diode_SMD:D_SMB"
 			(at 43.815 153.035 0)
 			(effects
@@
 			)
 		)
-		(property "Footprint" "Fuse:Fuse_0805_2012Metric"
+		(property "Footprint" "Fuse:Fuse_2512_6332Metric_Pad1.52x3.35mm_HandSolder"
 			(at 36.83 87.63 0)
 			(effects
@@
 			)
 		)
-		(property "Footprint" "Fuse:Fuse_0805_2012Metric"
+		(property "Footprint" "Fuse:Fuse_2512_6332Metric_Pad1.52x3.35mm_HandSolder"
 			(at 36.83 259.08 0)
 			(effects
@@
 			)
 		)
-		(property "Footprint" "Fuse:Fuse_0805_2012Metric"
+		(property "Footprint" "Fuse:Fuse_2512_6332Metric_Pad1.52x3.35mm_HandSolder"
 			(at 36.83 316.23 0)
 			(effects
@@
 			)
 		)
-		(property "Footprint" "Fuse:Fuse_0805_2012Metric"
+		(property "Footprint" "Fuse:Fuse_2512_6332Metric_Pad1.52x3.35mm_HandSolder"
 			(at 36.83 125.73 0)
 			(effects
@@
 			)
 		)
-		(property "Footprint" "Fuse:Fuse_2512_6332Metric_Pad1.52x3.35mm_HandSolder"
+		(property "Footprint" "Diode_SMD:D_SMB"
 			(at 43.815 114.935 0)
 			(effects
@@
 			)
 		)
-		(property "Footprint" "Fuse:Fuse_0805_2012Metric"
+		(property "Footprint" "Fuse:Fuse_2512_6332Metric_Pad1.52x3.35mm_HandSolder"
 			(at 36.83 144.78 0)
 			(effects
@@
 			)
 		)
-		(property "Footprint" "Fuse:Fuse_0805_2012Metric"
+		(property "Footprint" "Fuse:Fuse_2512_6332Metric_Pad1.52x3.35mm_HandSolder"
 			(at 36.83 220.98 0)
 			(effects
@@
 			)
 		)
-		(property "Footprint" "Fuse:Fuse_2512_6332Metric_Pad1.52x3.35mm_HandSolder"
+		(property "Footprint" "Diode_SMD:D_SMB"
 			(at 43.815 229.235 0)
 			(effects
@@
 			)
 		)
-		(property "Footprint" "Fuse:Fuse_2512_6332Metric_Pad1.52x3.35mm_HandSolder"
+		(property "Footprint" "Diode_SMD:D_SMB"
 			(at 43.815 133.985 0)
 			(effects
@@
 			)
 		)
-		(property "Footprint" "Fuse:Fuse_2512_6332Metric_Pad1.52x3.35mm_HandSolder"
+		(property "Footprint" "Diode_SMD:D_SMB"
 			(at 43.815 324.485 0)
 			(effects
@@
 			)
 		)
-		(property "Footprint" "Fuse:Fuse_2512_6332Metric_Pad1.52x3.35mm_HandSolder"
+		(property "Footprint" "Diode_SMD:D_SMB"
 			(at 43.815 191.135 0)
 			(effects
@@
 			)
 		)
-		(property "Footprint" "Fuse:Fuse_2512_6332Metric_Pad1.52x3.35mm_HandSolder"
+		(property "Footprint" "Diode_SMD:D_SMB"
 			(at 43.815 305.435 0)
 			(effects
@@
 			)
 		)
-		(property "Footprint" "Fuse:Fuse_0805_2012Metric"
+		(property "Footprint" "Fuse:Fuse_2512_6332Metric_Pad1.52x3.35mm_HandSolder"
 			(at 36.83 106.68 0)
 			(effects
@@
 			)
 		)
-		(property "Footprint" "Fuse:Fuse_2512_6332Metric_Pad1.52x3.35mm_HandSolder"
+		(property "Footprint" "Diode_SMD:D_SMB"
 			(at 43.815 172.085 0)
 			(effects
@@
 			)
 		)
-		(property "Footprint" "Fuse:Fuse_0805_2012Metric"
+		(property "Footprint" "Fuse:Fuse_2512_6332Metric_Pad1.52x3.35mm_HandSolder"
 			(at 36.83 354.33 0)
 			(effects
@@
 			)
 		)
-		(property "Footprint" "Fuse:Fuse_2512_6332Metric_Pad1.52x3.35mm_HandSolder"
+		(property "Footprint" "Diode_SMD:D_SMB"
 			(at 43.815 267.335 0)
 			(effects
@@
 			)
 		)
-		(property "Footprint" "Fuse:Fuse_0805_2012Metric"
+		(property "Footprint" "Fuse:Fuse_2512_6332Metric_Pad1.52x3.35mm_HandSolder"
 			(at 36.83 163.83 0)
 			(effects
@@
 			)
 		)
-		(property "Footprint" "Fuse:Fuse_0805_2012Metric"
+		(property "Footprint" "Fuse:Fuse_2512_6332Metric_Pad1.52x3.35mm_HandSolder"
 			(at 36.83 278.13 0)
 			(effects
@@
 			)
 		)
-		(property "Footprint" "Fuse:Fuse_0805_2012Metric"
+		(property "Footprint" "Fuse:Fuse_2512_6332Metric_Pad1.52x3.35mm_HandSolder"
 			(at 36.83 182.88 0)
 			(effects
